Commit message: Fix errors in Ubuntu 20.04

File: ids_description/urdf/jazzy_base.urdf.xacro (robot description, xacro)
@@ -15,9 +15,4 @@
     <xacro:property name="tip_m" value="0.1"/>
     <xacro:macro name="jazzy_base_macro">
-      <link name="world"/>
-      <joint name="joint_world_jazzy" type="floating">
-        <parent link="world"/>
-        <child link="link_jazzy"/>
-      </joint>
       <link name="link_jazzy">
         <visual>

File: ids_description/urdf/mrobot_1.urdf.xacro (robot description, xacro)
@@ -1,73 +1,74 @@
 <?xml version="1.0"?>
-<robot name="jazzy" xmlns:xacro="https://www.ros.org/wiki/xacro" >
-    <!--mobile base-->
-    <xacro:include filename="$(find ids_description)/urdf/wheeler_1.urdf.xacro" />
-    <xacro:wheel_base_macro>
-      <origin xyz="0 0 0" rpy="0 0 0"/>
-      <xacro:property name="friction_k" value="0.8"/>
-      <xacro:property name="friction_s" value="0.7"/>
-      <xacro:property name="chassis_x" value="0.7" />
-      <xacro:property name="chassis_y" value="0.4" />
-      <xacro:property name="chassis_z" value="0.1" />
-      <xacro:property name="chassis_m" value="40" />
-      <xacro:property name="wheel_r" value="0.11"/>
-      <xacro:property name="wheel_l" value="0.075"/>
-      <xacro:property name="wheel_m" value="0.5"/>
-      <xacro:property name="wheelbase" value="0.425" />
-      <xacro:property name="track" value="0.475" />
-      <xacro:property name="base_x" value="0.7" />
-      <xacro:property name="base_y" value="0.4" />
-      <xacro:property name="base_z" value="0.1" />
-      <xacro:property name="bumper_x" value="0.04" />
-      <xacro:property name="bumper_y" value="0.5" />
-      <xacro:property name="bumper_z" value="0.2" />
-    </xacro:wheel_base_macro>
-    <!--frame 3DOF-->
-    <xacro:include filename="$(find ids_description)/urdf/frame.urdf.xacro" />
-    <xacro:frame_macro parent="link_fbumper" name="mrobot">
-      <origin xyz="0.04 0 0.10" rpy="0 0 0"/>
-    </xacro:frame_macro>
-    <!--laser sensor-->
-    <xacro:include filename="$(find ids_description)/urdf/laser.urdf.xacro" />
-    <xacro:laser_macro parent="link_frame">
-      <xacro:property name="location_x" value="0.1"/>
-      <xacro:property name="location_y" value="0"/>
-      <xacro:property name="location_z" value="-0.1"/>
-    </xacro:laser_macro>
-    <!--RGB-D camera, look forward-->
-    <xacro:include filename="$(find ids_description)/urdf/realsense.urdf.xacro" />
-    <xacro:realsense_macro parent="link_hslider">
-      <xacro:property name="location_x" value="0.12"/>
-      <xacro:property name="location_y" value="0.0"/>
-      <xacro:property name="location_z" value="0.0325"/>
-      <xacro:property name="camera_width" value="640" />
-      <xacro:property name="camera_height" value="480" />
-      <xacro:property name="camera_name" value="rs435" />
-    </xacro:realsense_macro>
-    <!--camera, look backward-->
-    <xacro:include filename="$(find ids_description)/urdf/camera.urdf.xacro" />
-    <xacro:camera_macro parent="link_frame">
-      <xacro:property name="location_x" value="0.04"/>
-      <xacro:property name="location_y" value="0.0"/>
-      <xacro:property name="location_z" value="1.05"/>
-      <xacro:property name="location_r" value="3.14"/>
-      <xacro:property name="location_p" value="3.14"/>
-      <xacro:property name="location_y" value="0"/>
-      <xacro:property name="camera_width" value="640" />
-      <xacro:property name="camera_height" value="480" />
-      <xacro:property name="camera_name" value="back_cam" />
-    </xacro:camera_macro>
-    <!--camera, look upward-->
-    <xacro:include filename="$(find ids_description)/urdf/camera.urdf.xacro"/>
-    <xacro:camera_macro parent="link_tip">
-      <xacro:property name="location_x" value="0.02" />
-      <xacro:property name="location_y" value="0.0" />
-      <xacro:property name="location_z" value="0.015" />
-      <xacro:property name="location_r" value="0" />
-      <xacro:property name="location_p" value="-1.57" />
-      <xacro:property name="location_y" value="0" />
-      <xacro:property name="camera_width" value="640" />
-      <xacro:property name="camera_height" value="480" />
-      <xacro:property name="camera_name" value="cam_up"/>
-    </xacro:camera_macro>
+<!--mobile robot with indoor service device-->
+<robot name="robot" xmlns:xacro="https://www.ros.org/wiki/xacro" >
+  <!--mobile base-->
+  <xacro:include filename="$(find ids_description)/urdf/wheeler_1.urdf.xacro" />
+  <xacro:wheel_base_macro>
+    <origin xyz="0 0 0" rpy="0 0 0"/>
+    <xacro:property name="friction_k" value="0.8"/>
+    <xacro:property name="friction_s" value="0.7"/>
+    <xacro:property name="chassis_x" value="0.7" />
+    <xacro:property name="chassis_y" value="0.4" />
+    <xacro:property name="chassis_z" value="0.1" />
+    <xacro:property name="chassis_m" value="40" />
+    <xacro:property name="wheel_r" value="0.11"/>
+    <xacro:property name="wheel_l" value="0.075"/>
+    <xacro:property name="wheel_m" value="0.5"/>
+    <xacro:property name="wheelbase" value="0.425" />
+    <xacro:property name="track" value="0.475" />
+    <xacro:property name="base_x" value="0.7" />
+    <xacro:property name="base_y" value="0.4" />
+    <xacro:property name="base_z" value="0.1" />
+    <xacro:property name="bumper_x" value="0.04" />
+    <xacro:property name="bumper_y" value="0.5" />
+    <xacro:property name="bumper_z" value="0.2" />
+  </xacro:wheel_base_macro>
+  <!--frame 3DOF-->
+  <xacro:include filename="$(find ids_description)/urdf/frame.urdf.xacro" />
+  <xacro:frame_macro parent="link_fbumper" name="mrobot">
+    <origin xyz="0.04 0 0.10" rpy="0 0 0"/>
+  </xacro:frame_macro>
+  <!--laser sensor-->
+  <xacro:include filename="$(find ids_description)/urdf/laser.urdf.xacro" />
+  <xacro:laser_macro parent="link_frame">
+    <xacro:property name="location_x" value="0.1"/>
+    <xacro:property name="location_y" value="0"/>
+    <xacro:property name="location_z" value="-0.1"/>
+  </xacro:laser_macro>
+  <!--RGB-D camera, look forward-->
+  <xacro:include filename="$(find ids_description)/urdf/realsense.urdf.xacro" />
+  <xacro:realsense_macro parent="link_hslider">
+    <xacro:property name="location_x" value="0.12"/>
+    <xacro:property name="location_y" value="0.0"/>
+    <xacro:property name="location_z" value="0.0325"/>
+    <xacro:property name="camera_width" value="640" />
+    <xacro:property name="camera_height" value="480" />
+    <xacro:property name="camera_name" value="rs435" />
+  </xacro:realsense_macro>
+  <!--camera, look backward-->
+  <xacro:include filename="$(find ids_description)/urdf/camera.urdf.xacro" />
+  <xacro:camera_macro parent="link_frame">
+    <xacro:property name="location_x" value="0.04"/>
+    <xacro:property name="location_y" value="0.0"/>
+    <xacro:property name="location_z" value="1.05"/>
+    <xacro:property name="location_r" value="3.14"/>
+    <xacro:property name="location_p" value="3.14"/>
+    <xacro:property name="location_y" value="0"/>
+    <xacro:property name="camera_width" value="640" />
+    <xacro:property name="camera_height" value="480" />
+    <xacro:property name="camera_name" value="back_cam" />
+  </xacro:camera_macro>
+  <!--camera, look upward-->
+  <xacro:include filename="$(find ids_description)/urdf/camera.urdf.xacro"/>
+  <xacro:camera_macro parent="link_tip">
+    <xacro:property name="location_x" value="0.02" />
+    <xacro:property name="location_y" value="0.0" />
+    <xacro:property name="location_z" value="0.015" />
+    <xacro:property name="location_r" value="0" />
+    <xacro:property name="location_p" value="-1.57" />
+    <xacro:property name="location_y" value="0" />
+    <xacro:property name="camera_width" value="640" />
+    <xacro:property name="camera_height" value="480" />
+    <xacro:property name="camera_name" value="cam_up"/>
+  </xacro:camera_macro>
 </robot>

File: ids_description/urdf/wheeler_1.urdf.xacro (robot description, xacro)
@@ -1,3 +1,4 @@
 <?xml version="1.0" ?>
+<!--four wheel base-->
 <robot xmlns:xacro="https://www.ros.org/wiki/xacro" >
     <xacro:property name="friction_k" value="0.98"/>
@@ -11,6 +12,6 @@
     <xacro:property name="wheel_l" value="0.05"/>
     <xacro:property name="wheel_m" value="0.5"/>
-    <xacro:property name="wheelbase" value="0.25" /> <!--base on the wheel diameter and chassis_x-->
-    <xacro:property name="track" value="0.45" /> <!--base on the wheel width and chassis_y-->
+    <xacro:property name="wheelbase" value="0.25" />
+    <xacro:property name="track" value="0.45" />
     <xacro:property name="base_x" value="0.42" />
     <xacro:property name="base_y" value="0.4" />
@@ -23,11 +24,4 @@
     <xacro:property name="battery_m" value="20" />
     <xacro:macro name="wheel_base_macro" params="*origin">
-      <!-- Used for fixing robot to Gazebo 'base_link'-->
-      <link name="world"/>
-      <joint name="joint_world_chassis" type="floating">
-        <xacro:insert_block name="origin"/>
-        <parent link="world"/>
-        <child link="link_chassis"/>
-      </joint>
       <link name="link_chassis">
         <visual>

File: ids_description/urdf/wheeler_2.urdf.xacro (robot description, xacro)
@@ -24,10 +24,4 @@
     <!-- main triwheeler link -->
     <xacro:macro name="fourwheeler_base_macro">
-      <!-- Used for fixing robot to Gazebo 'base_link'-->
-      <link name="world"/>
-      <joint name="joint_world_chassis" type="floating">
-        <parent link="world"/>
-        <child link="link_chassis"/>
-      </joint>
       <link name="link_chassis">
         <visual>
