Commit message: support navigation

File: ids_description/urdf/laser.urdf.xacro (robot description, xacro)
@@ -16,5 +16,5 @@
           <origin xyz="0 0 0" rpy="0 0 0"/>
           <geometry>
-            <box size="0.05 0.05 0.05"/>
+            <box size="0.03 0.03 0.03"/>
           </geometry>
         </collision>
@@ -22,5 +22,5 @@
           <origin xyz="0 0 0" rpy="0 0 0"/>
           <geometry>
-            <box size="0.05 0.05 0.05"/>
+            <box size="0.03 0.03 0.03"/>
           </geometry>
         </visual>
@@ -48,12 +48,12 @@
             </scan>
             <range>
-              <min>0.01</min>
-              <max>100.0</max>
-              <resolution>0.005</resolution>
+              <min>0.05</min>
+              <max>30.0</max>
+              <resolution>0.01</resolution>
             </range>
             <noise>
               <type>gaussian</type>
               <mean>0.0</mean>
-              <stddev>0.001</stddev>
+              <stddev>0.01</stddev>
             </noise>
           </ray>

File: ids_description/urdf/mrobot_2.urdf.xacro (robot description, xacro)
@@ -34,3 +34,10 @@
       <xacro:property name="camera_name" value="cam_up"/>
     </xacro:camera_macro>
+    <!-- laser -->
+    <xacro:include filename="$(find ids_description)/urdf/laser.urdf.xacro"/>
+    <xacro:laser_macro parent="link_fbumper">
+      <xacro:property name="location_x" value="0.05" />
+      <xacro:property name="location_y" value="0" />
+      <xacro:property name="location_z" value="0" />
+    </xacro:laser_macro>
 </robot>

File: ids_description/urdf/wheeler_2.urdf.xacro (robot description, xacro)
@@ -258,11 +258,13 @@
           <wheelSeparation>${wheelbase}</wheelSeparation>
           <wheelDiameter>2*${wheel_r}</wheelDiameter>
+          <torque>30</torque>
+          <topicName>cmd_vel</topicName>
+          <commandTopic>cmd_vel</commandTopic>
           <robotBaseFrame>link_chassis</robotBaseFrame>
           <odometryFrame>odom</odometryFrame>
-          <torque>30</torque>
-          <topicName>cmd_vel</topicName>
+          <publish_odom>true</publish_odom>
+          <publish_odom_tf>false</publish_odom_tf>
           <odometryTopic>odom</odometryTopic>
           <broadcastTF>true</broadcastTF>
-          <commandTopic>cmd_vel</commandTopic>
           <covariance_x>0.0001</covariance_x>
           <covariance_y>0.0000</covariance_y>
