Commit message: auto charge support

File: ids_description/urdf/mrobot_2.urdf.xacro (robot description, xacro)
@@ -3,6 +3,6 @@
     <!--mobile base-->
     <xacro:include filename="$(find ids_description)/urdf/wheeler_2.urdf.xacro" />
-      <xacro:property name="friction_k" value="0.8"/>
-      <xacro:property name="friction_s" value="0.7"/>
+      <xacro:property name="friction_k" value="0.5"/>
+      <xacro:property name="friction_s" value="0.5"/>
     <xacro:fourwheeler_base_macro/>
     <!--frame 3DOF-->
