Commit message: revise code for self-plugging

File: ids_description/urdf/mrobot_1.urdf.xacro (robot description, xacro)
@@ -44,5 +44,5 @@
     <xacro:property name="camera_width" value="640" />
     <xacro:property name="camera_height" value="480" />
-    <xacro:property name="camera_name" value="rs435" />
+    <xacro:property name="camera_name" value="camera" />
   </xacro:realsense_macro>
   <!--camera, look backward-->
@@ -70,5 +70,5 @@
     <xacro:property name="camera_width" value="640" />
     <xacro:property name="camera_height" value="480" />
-    <xacro:property name="camera_name" value="cam_up"/>
+    <xacro:property name="camera_name" value="arducam"/>
   </xacro:camera_macro>
 </robot>

File: ids_description/urdf/mrobot_2.urdf.xacro (robot description, xacro)
@@ -19,5 +19,5 @@
       <xacro:property name="camera_width" value="640" />
       <xacro:property name="camera_height" value="480" />
-      <xacro:property name="camera_name" value="rs435" />
+      <xacro:property name="camera_name" value="camera" />
     </xacro:realsense_macro>
     <!--camera, look upward-->
@@ -32,5 +32,5 @@
       <xacro:property name="camera_width" value="600" />
       <xacro:property name="camera_height" value="600" />
-      <xacro:property name="camera_name" value="cam_up"/>
+      <xacro:property name="camera_name" value="arducam"/>
     </xacro:camera_macro>
     <!-- laser -->

File: ids_description/urdf/realsense.urdf.xacro (robot description, xacro)
@@ -68,5 +68,5 @@
             <imageTopicName>color/image_raw</imageTopicName>
             <cameraInfoTopicName>color/camera_info</cameraInfoTopicName>
-            <depthImageTopicName>depth/image_raw</depthImageTopicName>
+            <depthImageTopicName>depth/image_rect_raw</depthImageTopicName>
             <depthImageCameraInfoTopicName>depth/camera_info</depthImageCameraInfoTopicName>
             <pointCloudTopicName>depth/points</pointCloudTopicName>
