Commit message: Add new trained model which combines detection of all objets in one model

File: ids_description/urdf/frame.urdf.xacro (robot description, xacro)
@@ -97,5 +97,5 @@
         <child link="link_plug"/>
         <axis xyz="1 0 0"/>
-        <limit upper="0.1" lower="0" effort="300.0" velocity="0.1"/>
+        <limit upper="0.1" lower="0" effort="100.0" velocity="0.02"/>
       </joint>
       <link name="link_plug">

File: ids_description/urdf/mrobot_2.urdf.xacro (robot description, xacro)
@@ -14,7 +14,7 @@
     <xacro:include filename="$(find ids_description)/urdf/realsense.urdf.xacro" />
     <xacro:realsense_macro parent="link_hslider">
-      <xacro:property name="location_x" value="0.12"/>
+      <xacro:property name="location_x" value="0.06"/>
       <xacro:property name="location_y" value="0.0"/>
-      <xacro:property name="location_z" value="0.0325"/>
+      <xacro:property name="location_z" value="0.0725"/>
       <xacro:property name="camera_width" value="640" />
       <xacro:property name="camera_height" value="480" />

Commit message: change the effort and pid of each joint in frame.

File: ids_description/urdf/frame.urdf.xacro (robot description, xacro)
@@ -40,6 +40,5 @@
         <axis xyz="0 0 1"/>
         <limit upper="0.96" lower="0" effort="300.0" velocity="0.1"/>
-        <!-- <safety_controller k_velocity="3"/>
-        <dynamics damping="0" friction="0.0"/> -->
+        <dynamics damping="0" friction="30.0"/>
       </joint>
       <link name="link_vslider">
@@ -69,6 +68,5 @@
         <axis xyz="0 1 0"/>
         <limit upper="0.13" lower="-0.13" effort="300.0" velocity="0.1"/>
-        <!-- <safety_controller k_velocity="3"/>
-        <dynamics damping="0" friction="0.0"/> -->
+        <dynamics damping="0" friction="30.0"/>
       </joint>
       <link name="link_hslider">
@@ -97,5 +95,6 @@
         <child link="link_plug"/>
         <axis xyz="1 0 0"/>
-        <limit upper="0.1" lower="0" effort="100.0" velocity="0.02"/>
+        <limit upper="0.1" lower="0" effort="300.0" velocity="0.1"/>
+        <dynamics damping="0" friction="50.0"/>
       </joint>
       <link name="link_plug">
@@ -124,5 +123,5 @@
         <child link="link_hook"/>
         <axis xyz="0 -1 0"/>
-        <limit upper="1.48" lower="0" effort="300.0" velocity="0.1"/>
+        <limit upper="1.57" lower="0" effort="300.0" velocity="0.1"/>
       </joint>
       <link name="link_hook">

File: ids_description/urdf/mrobot_2.urdf.xacro (robot description, xacro)
@@ -3,6 +3,6 @@
     <!--mobile base-->
     <xacro:include filename="$(find ids_description)/urdf/wheeler_2.urdf.xacro" />
-      <xacro:property name="friction_k" value="0.5"/>
-      <xacro:property name="friction_s" value="0.5"/>
+      <xacro:property name="friction_k" value="0.98"/>
+      <xacro:property name="friction_s" value="0.98"/>
     <xacro:fourwheeler_base_macro/>
     <!--frame 3DOF-->

File: ids_description/urdf/wheeler_2.urdf.xacro (robot description, xacro)
@@ -7,5 +7,5 @@
     <xacro:property name="chassis_y" value="0.4" />
     <xacro:property name="chassis_z" value="0.05" />
-    <xacro:property name="chassis_m" value="28" />
+    <xacro:property name="chassis_m" value="40" />
     <xacro:property name="wheel_r" value="0.075"/>
     <xacro:property name="wheel_l" value="0.05"/>
@@ -16,5 +16,5 @@
     <xacro:property name="base_y" value="0.4" />
     <xacro:property name="base_z" value="0.075" />
-    <xacro:property name="base_m" value="2" />
+    <xacro:property name="base_m" value="20" />
     <xacro:property name="bumper_x" value="0.04" />
     <xacro:property name="bumper_y" value="0.46" />
@@ -258,5 +258,5 @@
           <wheelSeparation>${wheelbase}</wheelSeparation>
           <wheelDiameter>2*${wheel_r}</wheelDiameter>
-          <torque>30</torque>
+          <torque>200</torque>
           <topicName>cmd_vel</topicName>
           <commandTopic>cmd_vel</commandTopic>

Commit message: lock a joint in runtime

File: ids_description/urdf/frame.urdf.xacro (robot description, xacro)
@@ -96,5 +96,5 @@
         <axis xyz="1 0 0"/>
         <limit upper="0.1" lower="0" effort="300.0" velocity="0.1"/>
-        <dynamics damping="0" friction="50.0"/>
+        <dynamics damping="0" friction="30.0"/>
       </joint>
       <link name="link_plug">

Commit message: add contact sensor for plugged

File: ids_description/urdf/frame.urdf.xacro (robot description, xacro)
@@ -2,5 +2,5 @@
 <robot xmlns:xacro="https://www.ros.org/wiki/xacro" >
     <xacro:property name="PI" value="3.1415926535897931"/>
-    <xacro:property name="frame_m" value="2"/>
+    <xacro:property name="frame_m" value="20"/>
     <xacro:property name="vslider_m" value="2"/>
     <xacro:property name="hslider_m" value="1"/>
@@ -114,5 +114,32 @@
           <mass value="${plug_m}"/>
           <origin rpy="0 0 0" xyz="0.015 0 0"/>
-            <inertia ixx="${(1/12)*plug_m*(0.022*0.022+0.022*0.022)}" ixy="0" ixz="0" iyy="${(1/12)*plug_m*(0.022*0.022+0.07*0.07)}" iyz="0" izz="${(1/12)*plug_m*(0.07*0.07+0.022*0.022)}"/>
+          <inertia ixx="${(1/12)*plug_m*(0.022*0.022+0.022*0.022)}" ixy="0" ixz="0" iyy="${(1/12)*plug_m*(0.022*0.022+0.07*0.07)}" iyz="0" izz="${(1/12)*plug_m*(0.07*0.07+0.022*0.022)}"/>
+        </inertial>
+      </link>
+      <!--contact bumper-->
+      <joint name="joint_contact_bp" type="revolute">
+        <origin xyz="0.1405 0 0" rpy="0 0 0"/>
+        <parent link="link_plug"/>
+        <child link="link_contact_bp"/>
+        <axis xyz="1 0 0"/>
+        <limit upper="0" lower="0" effort="0.0" velocity="0.0"/>
+      </joint>
+      <link name="link_contact_bp">
+        <visual>
+          <origin rpy="0 0 0" xyz="0 0 0"/>
+          <geometry>
+            <box size="0.001 0.002 0.005"/>
+          </geometry>
+        </visual>
+        <collision name="bump_sensor_collision">
+          <origin rpy="0 0 0" xyz="0 0 0"/>
+          <geometry>
+            <box size="0.001 0.002 0.005"/>
+          </geometry>
+        </collision>
+        <inertial>
+          <mass value="0.01"/>
+          <origin rpy="0 0 0" xyz="0 0 0"/>
+          <inertia ixx="0.001" ixy="0" ixz="0" iyy="0.001" iyz="0" izz="0.001"/>
         </inertial>
       </link>
@@ -141,5 +168,5 @@
           <mass value="${hook_m}"/>
           <origin rpy="0 0 0" xyz="0.1 0 0"/>
-            <inertia ixx="${(1/3)*hook_m*(0.01*0.01+0.02*0.02)}" ixy="0" ixz="0" iyy="${(1/3)*hook_m*(4*0.2*0.2+0.01*0.01)}" iyz="0" izz="${(1/3)*hook_m*(4*0.2*0.2+0.02*0.02)}"/>
+          <inertia ixx="${(1/3)*hook_m*(0.01*0.01+0.02*0.02)}" ixy="0" ixz="0" iyy="${(1/3)*hook_m*(4*0.2*0.2+0.01*0.01)}" iyz="0" izz="${(1/3)*hook_m*(4*0.2*0.2+0.02*0.02)}"/>
         </inertial>
       </link>
@@ -165,5 +192,5 @@
           <mass value="${tip_m}"/>
           <origin rpy="0 0 0" xyz="0.01 0.02 0"/>
-            <inertia ixx="${(1/12)*tip_m*(0.06*0.06+0.01*0.01)}" ixy="0" ixz="0" iyy="${(1/3)*tip_m*(0.02*0.02+0.01*0.01)}" iyz="0" izz="${(1/12)*tip_m*(0.02*0.02+0.06*0.06)}"/>
+          <inertia ixx="${(1/12)*tip_m*(0.06*0.06+0.01*0.01)}" ixy="0" ixz="0" iyy="${(1/3)*tip_m*(0.02*0.02+0.01*0.01)}" iyz="0" izz="${(1/12)*tip_m*(0.02*0.02+0.06*0.06)}"/>
         </inertial>
       </link>
@@ -237,4 +264,7 @@
       <gazebo reference="link_tip">
         <material>Gazebo/Black</material>
+      </gazebo>
+      <gazebo reference="link_contact_bp">
+        <material>Gazebo/Blue</material>
       </gazebo>
       <!--force torque sensor-->
@@ -269,4 +299,17 @@
         </plugin>
       </gazebo>
+      <gazebo reference="link_contact_bp">
+        <sensor name="main_bumper" type="contact">
+          <contact>
+            <collision>link_contact_bp_fixed_joint_lump__bump_sensor_collision_collision</collision>
+          </contact>
+          <plugin name="gazebo_ros_bumper_controller" filename="libgazebo_ros_bumper.so">
+            <bumperTopicName>bumper_plug</bumperTopicName>
+            <frameName>world</frameName>
+            <alwaysOn>true</alwaysOn>
+            <updateRate>5.0</updateRate>
+          </plugin>
+        </sensor>
+      </gazebo>
     </xacro:macro>
 </robot>

Commit message: correct target position

File: ids_description/urdf/frame.urdf.xacro (robot description, xacro)
@@ -127,5 +127,5 @@
       <!--contact bumper-->
       <joint name="joint_contact_bp" type="revolute">
-        <origin xyz="0.1405 0 0" rpy="0 0 0"/>
+        <origin xyz="0.161 0 -0.00636" rpy="0 0 0"/>
         <parent link="link_plug"/>
         <child link="link_contact_bp"/>
@@ -137,5 +137,5 @@
           <origin rpy="0 0 0" xyz="0 0 0"/>
           <geometry>
-            <box size="0.001 0.002 0.005"/>
+            <box size="0.001 0.001 0.001"/>
           </geometry>
         </visual>
@@ -143,11 +143,11 @@
           <origin rpy="0 0 0" xyz="0 0 0"/>
           <geometry>
-            <box size="0.001 0.002 0.005"/>
-          </geometry>
-        </collision>
-        <inertial>
-          <mass value="0.01"/>
-          <origin rpy="0 0 0" xyz="0 0 0"/>
-          <inertia ixx="0.000000001" ixy="0" ixz="0" iyy="0.000000002" iyz="0" izz="0.000000001"/>
+            <box size="0.001 0.001 0.001"/>
+          </geometry>
+        </collision>
+        <inertial>
+          <mass value="0.001"/>
+          <origin rpy="0 0 0" xyz="0 0 0"/>
+          <inertia ixx="0.000000001" ixy="0" ixz="0" iyy="0.000000001" iyz="0" izz="0.000000001"/>
         </inertial>
       </link>
