Commit message: add kalman filter for filtering force signal

File: ids_description/urdf/base_square.urdf.xacro (robot description, xacro)
@@ -1,27 +1,28 @@
 <?xml version="1.0" ?>
-<!--four wheel base-->
 <robot xmlns:xacro="https://www.ros.org/wiki/xacro" >
-    <xacro:property name="friction_k" value="0.98"/>
-    <xacro:property name="friction_s" value="0.98"/>
+    <xacro:property name="mu" value="0.98"/>
+    <xacro:property name="mu2" value="0.98"/>
     <xacro:property name="PI" value="3.1415926535897931"/>
     <xacro:property name="chassis_x" value="0.42" />
     <xacro:property name="chassis_y" value="0.4" />
     <xacro:property name="chassis_z" value="0.05" />
-    <xacro:property name="chassis_m" value="28" />
+    <xacro:property name="chassis_m" value="40" />
     <xacro:property name="wheel_r" value="0.075"/>
     <xacro:property name="wheel_l" value="0.05"/>
     <xacro:property name="wheel_m" value="0.5"/>
-    <xacro:property name="wheelbase" value="0.25" />
-    <xacro:property name="track" value="0.45" />
+    <xacro:property name="wheelbase" value="0.25" /> <!--base on the wheel diameter and chassis_x-->
+    <xacro:property name="track" value="0.45" /> <!--base on the wheel width and chassis_y-->
     <xacro:property name="base_x" value="0.42" />
     <xacro:property name="base_y" value="0.4" />
     <xacro:property name="base_z" value="0.075" />
-    <xacro:property name="base_m" value="2" />
+    <xacro:property name="base_m" value="20" />
     <xacro:property name="bumper_x" value="0.04" />
-    <xacro:property name="bumper_y" value="0.5" />
+    <xacro:property name="bumper_y" value="0.46" />
     <xacro:property name="bumper_z" value="0.125" />
     <xacro:property name="bumper_m" value="1" />
-    <xacro:property name="battery_m" value="20" />
-    <xacro:macro name="wheel_base_macro" params="*origin">
+    <xacro:property name="battery_m" value="10" />
+    <xacro:property name="battery_l" value="0.1" />
+    <!-- main triwheeler link -->
+    <xacro:macro name="fourwheeler_base_macro">
       <link name="link_chassis">
         <visual>
@@ -229,13 +230,13 @@
       <link name="link_battery">
         <visual>
-          <origin xyz="-0.2 0 0.05" rpy="0 0 0" />
-          <geometry>
-            <box size="0.1 0.1 0.1"/>
-          </geometry>
-        </visual>
-        <collision>
-          <origin xyz="-0.2 0 0.05" rpy="0 0 0" />
-          <geometry>
-            <box size="0.1 0.1 0.1"/>
+          <origin xyz="-0.15 0 0.08" rpy="0 0 0" />
+          <geometry>
+            <box size="${battery_l} ${battery_l} ${battery_l}"/>
+          </geometry>
+        </visual>
+        <collision>
+          <origin xyz="-0.15 0 0.08" rpy="0 0 0" />
+          <geometry>
+            <box size="${battery_l} ${battery_l} ${battery_l}"/>
           </geometry>
         </collision>
@@ -243,5 +244,5 @@
           <mass value="${battery_m}"/>
           <origin rpy="0 0 0" xyz="0 0 0"/>
-          <inertia ixx="${(1/12)*battery_m*0.02}" ixy="0" ixz="0" iyy="${(1/12)*battery_m*0.02}" iyz="0" izz="${(1/12)*battery_m*0.02}"/>
+          <inertia ixx="${(1/12)*battery_m*(2*battery_l*battery_l)}" ixy="0" ixz="0" iyy="${(1/12)*battery_m*(2*battery_l*battery_l)}" iyz="0" izz="${(1/12)*battery_m*(2*battery_l*battery_l)}"/>
         </inertial>
       </link>
@@ -258,13 +259,16 @@
           <wheelSeparation>${wheelbase}</wheelSeparation>
           <wheelDiameter>2*${wheel_r}</wheelDiameter>
+          <torque>30</torque>
+          <topicName>cmd_vel</topicName>
+          <commandTopic>cmd_vel</commandTopic>
           <robotBaseFrame>link_chassis</robotBaseFrame>
           <odometryFrame>odom</odometryFrame>
-          <torque>30</torque>
+          <publish_odom>true</publish_odom>
+          <publish_odom_tf>false</publish_odom_tf>
           <odometryTopic>odom</odometryTopic>
           <broadcastTF>true</broadcastTF>
-          <commandTopic>cmd_vel</commandTopic>
-          <covariance_x>0.001</covariance_x>
-          <covariance_y>0.001</covariance_y>
-          <covariance_yaw>0.001</covariance_yaw>
+          <covariance_x>0.0001</covariance_x>
+          <covariance_y>0.0000</covariance_y>
+          <covariance_yaw>0.01</covariance_yaw>
         </plugin>
       </gazebo>
@@ -281,25 +285,22 @@
         <material>Gazebo/DarkGrey</material>
       </gazebo>
-      <gazebo reference="link_battery">
-        <material>Gazebo/Grey</material>
-      </gazebo>
       <gazebo reference="link_lrwheel">
-        <mu1>${friction_k}</mu1>
-        <mu2>${friction_s}</mu2>
+        <mu1>${mu}</mu1>
+        <mu2>${mu2}</mu2>
         <material>Gazebo/Black</material>
       </gazebo>
       <gazebo reference="link_rrwheel">
-        <mu1>${friction_k}</mu1>
-        <mu2>${friction_s}</mu2>
+        <mu1>${mu}</mu1>
+        <mu2>${mu2}</mu2>
         <material>Gazebo/Black</material>
       </gazebo>
       <gazebo reference="link_lfwheel">
-        <mu1>${friction_k}</mu1>
-        <mu2>${friction_s}</mu2>
+        <mu1>${mu}</mu1>
+        <mu2>${mu2}</mu2>
         <material>Gazebo/Black</material>
       </gazebo>
       <gazebo reference="link_rfwheel">
-        <mu1>${friction_k}</mu1>
-        <mu2>${friction_s}</mu2>
+        <mu1>${mu}</mu1>
+        <mu2>${mu2}</mu2>
         <material>Gazebo/Black</material>
       </gazebo>

File: ids_description/urdf/frame.urdf.xacro (robot description, xacro)
@@ -4,8 +4,8 @@
     <xacro:property name="frame_m" value="20"/>
     <xacro:property name="vslider_m" value="2"/>
-    <xacro:property name="hslider_m" value="1"/>
-    <xacro:property name="plug_m" value="0.5"/>
-    <xacro:property name="hook_m" value="0.2"/>
-    <xacro:property name="tip_m" value="0.1"/>
+    <xacro:property name="hslider_m" value="0.8"/>
+    <xacro:property name="plug_m" value="0.2"/>
+    <xacro:property name="hook_m" value="0.5"/>
+    <xacro:property name="tip_m" value="0.2"/>
     <xacro:macro name="frame_macro" params="parent name *origin">
       <joint name="joint_jazzy_frame" type="fixed">
@@ -39,6 +39,6 @@
         <child link="link_vslider"/>
         <axis xyz="0 0 1"/>
-        <limit upper="0.96" lower="0" effort="300.0" velocity="0.1"/>
-        <dynamics damping="0" friction="30.0"/>
+        <limit upper="0.96" lower="0" effort="100.0" velocity="0.1"/>
+        <dynamics damping="0" friction="5.0"/>
       </joint>
       <link name="link_vslider">
@@ -67,6 +67,6 @@
         <child link="link_hslider"/>
         <axis xyz="0 1 0"/>
-        <limit upper="0.13" lower="-0.13" effort="300.0" velocity="0.1"/>
-        <dynamics damping="0" friction="30.0"/>
+        <limit upper="0.13" lower="-0.13" effort="100.0" velocity="0.1"/>
+        <dynamics damping="0" friction="5.0"/>
       </joint>
       <link name="link_hslider">
@@ -95,6 +95,6 @@
         <child link="link_plug"/>
         <axis xyz="1 0 0"/>
-        <limit upper="0.1" lower="0" effort="300.0" velocity="0.1"/>
-        <dynamics damping="0" friction="30.0"/>
+        <limit upper="0.1" lower="0" effort="100.0" velocity="0.1"/>
+        <dynamics damping="0" friction="5.0"/>
       </joint>
       <link name="link_plug">
@@ -110,4 +110,12 @@
             <mesh filename="package://ids_description/meshes/jazzy/plug.obj" scale="0.01 0.01 0.01"/>
           </geometry>
+          <surface>
+            <friction>
+              <ode>
+                <mu>0.01</mu>
+                <mu2>0.01</mu2>
+              </ode>
+            </friction>
+          </surface>
         </collision>
         <inertial>
@@ -141,5 +149,5 @@
           <mass value="0.01"/>
           <origin rpy="0 0 0" xyz="0 0 0"/>
-          <inertia ixx="0.001" ixy="0" ixz="0" iyy="0.001" iyz="0" izz="0.001"/>
+          <inertia ixx="0.000000001" ixy="0" ixz="0" iyy="0.000000002" iyz="0" izz="0.000000001"/>
         </inertial>
       </link>
@@ -164,4 +172,12 @@
             <box size="0.25 0.02 0.01"/>
           </geometry>
+          <surface>
+            <friction>
+              <ode>
+                <mu>0.01</mu>
+                <mu2>0.01</mu2>
+              </ode>
+            </friction>
+          </surface>
         </collision>
         <inertial>
@@ -268,5 +284,5 @@
         <material>Gazebo/Blue</material>
       </gazebo>
-      <!--force torque sensor-->
+      <!--sensors-->
       <gazebo reference="joint_frame_hook">
         <provideFeedback>true</provideFeedback>
@@ -276,7 +292,7 @@
       </gazebo>
       <gazebo>
-        <plugin name="ft_sensor" filename="libgazebo_ros_ft_sensor.so">
+        <plugin name="sidebar_force_sensor" filename="libgazebo_ros_ft_sensor.so">
           <updateRate>100.0</updateRate>
-          <topicName>tf_sensor_hook</topicName>
+          <topicName>ft_sidebar</topicName>
           <jointName>joint_frame_hook</jointName>
           <noise>
@@ -288,7 +304,7 @@
       </gazebo>
       <gazebo>
-        <plugin name="ft_sensor" filename="libgazebo_ros_ft_sensor.so">
+        <plugin name="endeffector_force_sensor" filename="libgazebo_ros_ft_sensor.so">
           <updateRate>100.0</updateRate>
-          <topicName>tf_sensor_slider</topicName>
+          <topicName>ft_endeffector</topicName>
           <jointName>joint_vslider_hslider</jointName>
           <noise>

File: ids_description/urdf/mrobot.urdf.xacro (robot description, xacro)
@@ -2,7 +2,7 @@
 <robot name="jazzy" xmlns:xacro="https://www.ros.org/wiki/xacro" >
     <!--mobile base-->
-    <xacro:include filename="$(find ids_description)/urdf/wheeler_2.urdf.xacro" />
-      <xacro:property name="friction_k" value="0.98"/>
-      <xacro:property name="friction_s" value="0.98"/>
+    <xacro:include filename="$(find ids_description)/urdf/base_square.urdf.xacro" />
+      <xacro:property name="mu" value="0.9"/>
+      <xacro:property name="mu2" value="0.7"/>
     <xacro:fourwheeler_base_macro/>
     <!--frame 3DOF-->

Commit message: change physic engine config for door opening simulation

File: ids_description/urdf/base_square.urdf.xacro (robot description, xacro)
@@ -7,5 +7,5 @@
     <xacro:property name="chassis_y" value="0.4" />
     <xacro:property name="chassis_z" value="0.05" />
-    <xacro:property name="chassis_m" value="40" />
+    <xacro:property name="chassis_m" value="28" />
     <xacro:property name="wheel_r" value="0.075"/>
     <xacro:property name="wheel_l" value="0.05"/>
@@ -16,5 +16,5 @@
     <xacro:property name="base_y" value="0.4" />
     <xacro:property name="base_z" value="0.075" />
-    <xacro:property name="base_m" value="20" />
+    <xacro:property name="base_m" value="5" />
     <xacro:property name="bumper_x" value="0.04" />
     <xacro:property name="bumper_y" value="0.46" />
