Commit message: update parameters of navigation

File: ids_description/urdf/base_square.urdf.xacro (robot description, xacro)
@@ -1,308 +1,306 @@
 <?xml version="1.0" ?>
-<robot xmlns:xacro="https://www.ros.org/wiki/xacro" >
-    <xacro:property name="mu" value="0.98"/>
-    <xacro:property name="mu2" value="0.98"/>
-    <xacro:property name="PI" value="3.1415926535897931"/>
-    <xacro:property name="chassis_x" value="0.42" />
-    <xacro:property name="chassis_y" value="0.4" />
-    <xacro:property name="chassis_z" value="0.05" />
-    <xacro:property name="chassis_m" value="28" />
-    <xacro:property name="wheel_r" value="0.075"/>
-    <xacro:property name="wheel_l" value="0.05"/>
-    <xacro:property name="wheel_m" value="0.5"/>
-    <xacro:property name="wheelbase" value="0.25" /> <!--base on the wheel diameter and chassis_x-->
-    <xacro:property name="track" value="0.45" /> <!--base on the wheel width and chassis_y-->
-    <xacro:property name="base_x" value="0.42" />
-    <xacro:property name="base_y" value="0.4" />
-    <xacro:property name="base_z" value="0.075" />
-    <xacro:property name="base_m" value="5" />
-    <xacro:property name="bumper_x" value="0.04" />
-    <xacro:property name="bumper_y" value="0.46" />
-    <xacro:property name="bumper_z" value="0.125" />
-    <xacro:property name="bumper_m" value="1" />
-    <xacro:property name="battery_m" value="10" />
-    <xacro:property name="battery_l" value="0.1" />
-    <!-- main triwheeler link -->
-    <xacro:macro name="fourwheeler_base_macro">
-      <link name="link_chassis">
-        <visual>
-          <origin xyz="0 0 0" rpy="0 0 0" />
-          <geometry>
-            <box size="${chassis_x} ${chassis_y} ${chassis_z}"/>
-          </geometry>
-        </visual>
-        <collision>
-          <origin xyz="0 0 0" rpy="0 0 0" />
-          <geometry>
-            <box size="${chassis_x} ${chassis_y} ${chassis_z}"/>
-          </geometry>
-        </collision>
-        <inertial>
-          <mass value="${chassis_m}"/>
-          <origin rpy="0 0 0" xyz="0 0 0"/>
-          <inertia ixx="${(1/12)*chassis_m*(chassis_y*chassis_y+chassis_z*chassis_z)}" ixy="0" ixz="0" iyy="${(1/12)*chassis_m*(chassis_z*chassis_z+chassis_x*chassis_x)}" iyz="0" izz="${(1/12)*chassis_m*(chassis_x*chassis_x+chassis_y*chassis_y)}"/>
-        </inertial>
-      </link>
-      <!--left rear wheel-->
-      <joint name="joint_chassis_lrwheel" type="continuous">
-        <origin xyz="-${wheelbase/2} ${track/2} 0" rpy="0 0 0" />
-        <parent link="link_chassis"/>
-        <child link="link_lrwheel"/>
-        <axis xyz="0 1 0" rpy="0 0 0" />
-      </joint>
-      <link name="link_lrwheel">
-        <visual>
-          <origin rpy="${PI/2} 0 0" xyz="0 0 0"/>
-          <geometry>
-            <cylinder length="${wheel_l}" radius="${wheel_r}"/>
-          </geometry>
-        </visual>
-        <collision>
-          <origin rpy="${PI/2} 0 0" xyz="0 0 0" />
-          <geometry>
-            <cylinder length="${wheel_l}" radius="${wheel_r}"/>
-          </geometry>
-        </collision>
-        <inertial>
-          <mass value="${wheel_m}"/>
-          <origin rpy="${PI/2} 0 0" xyz="0 0 0"/>
-          <inertia ixx="${(1/12)*wheel_m*(3*wheel_r*wheel_r+wheel_l*wheel_l)}" ixy="0" ixz="0" iyy="${(1/12)*wheel_m*(3*wheel_r*wheel_r+wheel_l*wheel_l)}" iyz="0" izz="${(1/2)*wheel_m*wheel_r*wheel_r}"/>
-        </inertial>
-      </link>
-      <!--right rear wheel-->
-      <joint name="joint_chassis_rrwheel" type="continuous">
-        <origin xyz="-${wheelbase/2} -${track/2} 0" rpy="0 0 0" />
-        <parent link="link_chassis"/>
-        <child link="link_rrwheel"/>
-        <axis xyz="0 1 0" rpy="0 0 0" />
-      </joint>
-      <link name="link_rrwheel">
-        <visual>
-          <origin rpy="${PI/2} 0 0" xyz="0 0 0"/>
-          <geometry>
-            <cylinder length="${wheel_l}" radius="${wheel_r}"/>
-          </geometry>
-        </visual>
-        <collision>
-          <origin rpy="${PI/2} 0 0" xyz="0 0 0" />
-          <geometry>
-            <cylinder length="${wheel_l}" radius="${wheel_r}"/>
-          </geometry>
-        </collision>
-        <inertial>
-          <mass value="${wheel_m}"/>
-          <origin rpy="${PI/2} 0 0" xyz="0 0 0"/>
-          <inertia ixx="${(1/12)*wheel_m*(3*wheel_r*wheel_r+wheel_l*wheel_l)}" ixy="0" ixz="0" iyy="${(1/12)*wheel_m*(3*wheel_r*wheel_r+wheel_l*wheel_l)}" iyz="0" izz="${(1/2)*wheel_m*wheel_r*wheel_r}"/>
-        </inertial>
-      </link>
-      <!--left front wheel-->
-      <joint name="joint_chassis_lfwheel" type="continuous">
-        <origin xyz="${wheelbase/2} ${track/2} 0" rpy="0 0 0" />
-        <parent link="link_chassis"/>
-        <child link="link_lfwheel"/>
-        <axis xyz="0 1 0" rpy="0 0 0" />
-      </joint>
-      <link name="link_lfwheel">
-        <visual>
-          <origin rpy="${PI/2} 0 0" xyz="0 0 0"/>
-          <geometry>
-            <cylinder length="${wheel_l}" radius="${wheel_r}"/>
-          </geometry>
-        </visual>
-        <collision>
-          <origin rpy="${PI/2} 0 0" xyz="0 0 0" />
-          <geometry>
-            <cylinder length="${wheel_l}" radius="${wheel_r}"/>
-          </geometry>
-        </collision>
-        <inertial>
-          <mass value="${wheel_m}"/>
-          <origin rpy="${PI/2} 0 0" xyz="0 0 0"/>
-          <inertia ixx="${(1/12)*wheel_m*(3*wheel_r*wheel_r+wheel_l*wheel_l)}" ixy="0" ixz="0" iyy="${(1/12)*wheel_m*(3*wheel_r*wheel_r+wheel_l*wheel_l)}" iyz="0" izz="${(1/2)*wheel_m*wheel_r*wheel_r}"/>
-        </inertial>
-      </link>
-      <!--right front wheel-->
-      <joint name="joint_chassis_rfwheel" type="continuous">
-        <origin xyz="${wheelbase/2} -${track/2} 0" rpy="0 0 0" />
-        <parent link="link_chassis"/>
-        <child link="link_rfwheel"/>
-        <axis xyz="0 1 0" rpy="0 0 0" />
-      </joint>
-      <link name="link_rfwheel">
-        <visual>
-          <origin rpy="${PI/2} 0 0" xyz="0 0 0"/>
-          <geometry>
-            <cylinder length="${wheel_l}" radius="${wheel_r}"/>
-          </geometry>
-        </visual>
-        <collision>
-          <origin rpy="${PI/2} 0 0" xyz="0 0 0" />
-          <geometry>
-            <cylinder length="${wheel_l}" radius="${wheel_r}"/>
-          </geometry>
-        </collision>
-        <inertial>
-          <mass value="${wheel_m}"/>
-          <origin rpy="${PI/2} 0 0" xyz="0 0 0"/>
-          <inertia ixx="${(1/12)*wheel_m*(3*wheel_r*wheel_r+wheel_l*wheel_l)}" ixy="0" ixz="0" iyy="${(1/12)*wheel_m*(3*wheel_r*wheel_r+wheel_l*wheel_l)}" iyz="0" izz="${(1/2)*wheel_m*wheel_r*wheel_r}"/>
-        </inertial>
-      </link>
-      <!--upper base-->
-      <joint name="joint_chassis_base" type="fixed">
-        <origin xyz="0 0 ${chassis_z/2}" rpy="0 0 0"/>
-        <parent link="link_chassis"/>
-        <child link="link_base"/>
-      </joint>
-      <link name="link_base">
-        <visual>
-          <origin xyz="0 0 ${base_z/2}" rpy="0 0 0" />
-          <geometry>
-            <box size="${base_x} ${base_y} ${base_z}"/>
-          </geometry>
-        </visual>
-        <collision>
-          <origin xyz="0 0 ${base_z/2}" rpy="0 0 0" />
-          <geometry>
-            <box size="${base_x} ${base_y} ${base_z}"/>
-          </geometry>
-        </collision>
-        <inertial>
-          <mass value="${base_m}"/>
-          <origin rpy="0 0 0" xyz="0 0 0"/>
-          <inertia ixx="${(1/12)*base_m*(base_y*base_y+base_z*base_z)}" ixy="0" ixz="0" iyy="${(1/12)*base_m*(base_z*base_z+base_x*base_x)}" iyz="0" izz="${(1/12)*base_m*(base_x*base_x+base_y*base_y)}"/>
-        </inertial>
-      </link>
-      <!--bumper-->
-      <joint name="joint_chassis_fbumper" type="fixed">
-        <origin xyz="${chassis_x/2} 0 ${(chassis_z+base_z)/2-chassis_z/2}" rpy="0 0 0"/>
-        <parent link="link_chassis"/>
-        <child link="link_fbumper"/>
-      </joint>
-      <link name="link_fbumper">
-        <visual>
-          <origin xyz="${bumper_x/2} 0 0" rpy="0 0 0" />
-          <geometry>
-            <box size="${bumper_x} ${bumper_y} ${bumper_z}"/>
-          </geometry>
-        </visual>
-        <collision>
-          <origin xyz="${bumper_x/2} 0 0" rpy="0 0 0" />
-          <geometry>
-            <box size="${bumper_x} ${bumper_y} ${bumper_z}"/>
-          </geometry>
-        </collision>
-        <inertial>
-          <mass value="${bumper_m}"/>
-          <origin rpy="0 0 0" xyz="0 0 0"/>
-          <inertia ixx="${(1/12)*bumper_m*(bumper_y*bumper_y+bumper_z*bumper_z)}" ixy="0" ixz="0" iyy="${(1/12)*bumper_m*(bumper_z*bumper_z+bumper_x*bumper_x)}" iyz="0" izz="${(1/12)*bumper_m*(bumper_x*bumper_x+bumper_y*bumper_y)}"/>
-        </inertial>
-      </link>
-      <joint name="joint_chassis_rbumper" type="fixed">
-        <origin xyz="-${chassis_x/2} 0 ${(chassis_z+base_z)/2-chassis_z/2}" rpy="0 0 0"/>
-        <parent link="link_chassis"/>
-        <child link="link_rbumper"/>
-      </joint>
-      <link name="link_rbumper">
-        <visual>
-          <origin xyz="-${bumper_x/2} 0 0" rpy="0 0 0" />
-          <geometry>
-            <box size="${bumper_x} ${bumper_y} ${bumper_z}"/>
-          </geometry>
-        </visual>
-        <collision>
-          <origin xyz="-${bumper_x/2} 0 0" rpy="0 0 0" />
-          <geometry>
-            <box size="${bumper_x} ${bumper_y} ${bumper_z}"/>
-          </geometry>
-        </collision>
-        <inertial>
-          <mass value="${bumper_m}"/>
-          <origin rpy="0 0 0" xyz="0 0 0"/>
-          <inertia ixx="${(1/12)*bumper_m*(bumper_y*bumper_y+bumper_z*bumper_z)}" ixy="0" ixz="0" iyy="${(1/12)*bumper_m*(bumper_z*bumper_z+bumper_x*bumper_x)}" iyz="0" izz="${(1/12)*bumper_m*(bumper_x*bumper_x+bumper_y*bumper_y)}"/>
-        </inertial>
-      </link>
-      <!--baterry-->
-      <joint name="joint_base_battery" type="fixed">
-        <origin xyz="0 0 ${base_z/2}" rpy="0 0 0"/>
-        <parent link="link_base"/>
-        <child link="link_battery"/>
-      </joint>
-      <link name="link_battery">
-        <visual>
-          <origin xyz="-0.15 0 0.08" rpy="0 0 0" />
-          <geometry>
-            <box size="${battery_l} ${battery_l} ${battery_l}"/>
-          </geometry>
-        </visual>
-        <collision>
-          <origin xyz="-0.15 0 0.08" rpy="0 0 0" />
-          <geometry>
-            <box size="${battery_l} ${battery_l} ${battery_l}"/>
-          </geometry>
-        </collision>
-        <inertial>
-          <mass value="${battery_m}"/>
-          <origin rpy="0 0 0" xyz="0 0 0"/>
-          <inertia ixx="${(1/12)*battery_m*(2*battery_l*battery_l)}" ixy="0" ixz="0" iyy="${(1/12)*battery_m*(2*battery_l*battery_l)}" iyz="0" izz="${(1/12)*battery_m*(2*battery_l*battery_l)}"/>
-        </inertial>
-      </link>
-      <!--Gazebo-->
-      <!-- skid steering controller -->
-      <gazebo>
-        <plugin name="skid_steer_drive_controller" filename="libgazebo_ros_skid_steer_drive.so">
-          <updateRate>100.0</updateRate>
-          <robotNamespace>/</robotNamespace>
-          <leftFrontJoint>joint_chassis_lfwheel</leftFrontJoint>
-          <rightFrontJoint>joint_chassis_rfwheel</rightFrontJoint>
-          <leftRearJoint>joint_chassis_lrwheel</leftRearJoint>
-          <rightRearJoint>joint_chassis_rrwheel</rightRearJoint>
-          <wheelSeparation>${wheelbase}</wheelSeparation>
-          <wheelDiameter>2*${wheel_r}</wheelDiameter>
-          <torque>30</torque>
-          <topicName>cmd_vel</topicName>
-          <commandTopic>cmd_vel</commandTopic>
-          <robotBaseFrame>link_chassis</robotBaseFrame>
-          <odometryFrame>odom</odometryFrame>
-          <publish_odom>true</publish_odom>
-          <publish_odom_tf>false</publish_odom_tf>
-          <odometryTopic>odom</odometryTopic>
-          <broadcastTF>true</broadcastTF>
-          <covariance_x>0.0001</covariance_x>
-          <covariance_y>0.0000</covariance_y>
-          <covariance_yaw>0.01</covariance_yaw>
-        </plugin>
-      </gazebo>
-      <gazebo reference="link_chassis">
-        <material>Gazebo/Grey</material>
-      </gazebo>
-      <gazebo reference="link_base">
-        <material>Gazebo/DarkGrey</material>
-      </gazebo>
-      <gazebo reference="link_fbumper">
-        <material>Gazebo/DarkGrey</material>
-      </gazebo>
-      <gazebo reference="link_rbumper">
-        <material>Gazebo/DarkGrey</material>
-      </gazebo>
-      <gazebo reference="link_lrwheel">
-        <mu1>${mu}</mu1>
-        <mu2>${mu2}</mu2>
-        <material>Gazebo/Black</material>
-      </gazebo>
-      <gazebo reference="link_rrwheel">
-        <mu1>${mu}</mu1>
-        <mu2>${mu2}</mu2>
-        <material>Gazebo/Black</material>
-      </gazebo>
-      <gazebo reference="link_lfwheel">
-        <mu1>${mu}</mu1>
-        <mu2>${mu2}</mu2>
-        <material>Gazebo/Black</material>
-      </gazebo>
-      <gazebo reference="link_rfwheel">
-        <mu1>${mu}</mu1>
-        <mu2>${mu2}</mu2>
-        <material>Gazebo/Black</material>
-      </gazebo>
-    </xacro:macro>
+<robot xmlns:xacro="https://www.ros.org/wiki/xacro">
+  <xacro:property name="mu" value="0.98"/>
+  <xacro:property name="mu2" value="0.98"/>
+  <xacro:property name="PI" value="3.1415926535897931"/>
+  <xacro:property name="chassis_x" value="0.42" />
+  <xacro:property name="chassis_y" value="0.4" />
+  <xacro:property name="chassis_z" value="0.05" />
+  <xacro:property name="chassis_m" value="28" />
+  <xacro:property name="wheel_r" value="0.075"/>
+  <xacro:property name="wheel_l" value="0.05"/>
+  <xacro:property name="wheel_m" value="0.5"/>
+  <xacro:property name="wheelbase" value="0.25" /> <!--base on the wheel diameter and chassis_x-->
+  <xacro:property name="track" value="0.45" /> <!--base on the wheel width and chassis_y-->
+  <xacro:property name="base_x" value="0.42" />
+  <xacro:property name="base_y" value="0.4" />
+  <xacro:property name="base_z" value="0.075" />
+  <xacro:property name="base_m" value="5" />
+  <xacro:property name="bumper_x" value="0.04" />
+  <xacro:property name="bumper_y" value="0.46" />
+  <xacro:property name="bumper_z" value="0.125" />
+  <xacro:property name="bumper_m" value="1" />
+  <xacro:property name="battery_m" value="10" />
+  <xacro:property name="battery_l" value="0.1" />
+  <!-- main triwheeler link -->
+  <xacro:macro name="fourwheeler_base_macro">
+    <link name="link_chassis">
+      <visual>
+        <origin xyz="0 0 0" rpy="0 0 0" />
+        <geometry>
+          <box size="${chassis_x} ${chassis_y} ${chassis_z}"/>
+        </geometry>
+      </visual>
+      <collision>
+        <origin xyz="0 0 0" rpy="0 0 0" />
+        <geometry>
+          <box size="${chassis_x} ${chassis_y} ${chassis_z}"/>
+        </geometry>
+      </collision>
+      <inertial>
+        <mass value="${chassis_m}"/>
+        <origin rpy="0 0 0" xyz="0 0 0"/>
+        <inertia ixx="${(1/12)*chassis_m*(chassis_y*chassis_y+chassis_z*chassis_z)}" ixy="0" ixz="0" iyy="${(1/12)*chassis_m*(chassis_z*chassis_z+chassis_x*chassis_x)}" iyz="0" izz="${(1/12)*chassis_m*(chassis_x*chassis_x+chassis_y*chassis_y)}"/>
+      </inertial>
+    </link>
+    <!--left rear wheel-->
+    <joint name="joint_chassis_lrwheel" type="continuous">
+      <origin xyz="-${wheelbase/2} ${track/2} 0" rpy="0 0 0" />
+      <parent link="link_chassis"/>
+      <child link="link_lrwheel"/>
+      <axis xyz="0 1 0" rpy="0 0 0" />
+    </joint>
+    <link name="link_lrwheel">
+      <visual>
+        <origin rpy="${PI/2} 0 0" xyz="0 0 0"/>
+        <geometry>
+          <cylinder length="${wheel_l}" radius="${wheel_r}"/>
+        </geometry>
+      </visual>
+      <collision>
+        <origin rpy="${PI/2} 0 0" xyz="0 0 0" />
+        <geometry>
+          <cylinder length="${wheel_l}" radius="${wheel_r}"/>
+        </geometry>
+      </collision>
+      <inertial>
+        <mass value="${wheel_m}"/>
+        <origin rpy="${PI/2} 0 0" xyz="0 0 0"/>
+        <inertia ixx="${(1/12)*wheel_m*(3*wheel_r*wheel_r+wheel_l*wheel_l)}" ixy="0" ixz="0" iyy="${(1/12)*wheel_m*(3*wheel_r*wheel_r+wheel_l*wheel_l)}" iyz="0" izz="${(1/2)*wheel_m*wheel_r*wheel_r}"/>
+      </inertial>
+    </link>
+    <!--right rear wheel-->
+    <joint name="joint_chassis_rrwheel" type="continuous">
+      <origin xyz="-${wheelbase/2} -${track/2} 0" rpy="0 0 0" />
+      <parent link="link_chassis"/>
+      <child link="link_rrwheel"/>
+      <axis xyz="0 1 0" rpy="0 0 0" />
+    </joint>
+    <link name="link_rrwheel">
+      <visual>
+        <origin rpy="${PI/2} 0 0" xyz="0 0 0"/>
+        <geometry>
+          <cylinder length="${wheel_l}" radius="${wheel_r}"/>
+        </geometry>
+      </visual>
+      <collision>
+        <origin rpy="${PI/2} 0 0" xyz="0 0 0" />
+        <geometry>
+          <cylinder length="${wheel_l}" radius="${wheel_r}"/>
+        </geometry>
+      </collision>
+      <inertial>
+        <mass value="${wheel_m}"/>
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
File: ids_description/urdf/camera.urdf.xacro (robot description, xacro)
@@ -61,9 +61,9 @@
         <plugin name="camera_controller" filename="libgazebo_ros_camera.so">
           <alwaysOn>true</alwaysOn>
-          <updateRate>0.0</updateRate>
-          <cameraName>${camera_name}</cameraName>
+          <updateRate>60</updateRate>
+          <cameraName>/$(arg ns)/${camera_name}</cameraName>
           <imageTopicName>image</imageTopicName>
           <cameraInfoTopicName>camera_info</cameraInfoTopicName>
-          <frameName>${camera_name}</frameName>
+          <frameName>$(arg tf_prefix)/${camera_name}</frameName>
           <hackBaseline>0.07</hackBaseline>
           <distortionK1>0.0</distortionK1>

File: ids_description/urdf/frame.urdf.xacro (robot description, xacro)
@@ -8,5 +8,5 @@
     <xacro:property name="hook_m" value="0.5"/>
     <xacro:property name="tip_m" value="0.2"/>
-    <xacro:macro name="frame_macro" params="parent name *origin">
+    <xacro:macro name="frame_macro" params="parent *origin">
       <joint name="joint_jazzy_frame" type="fixed">
         <xacro:insert_block name="origin"/>
@@ -254,7 +254,7 @@
       <gazebo>
         <plugin name="gazebo_ros_control" filename="libgazebo_ros_control.so">
-          <robotNamespace>/${name}</robotNamespace>
           <robotSimType>gazebo_ros_control/DefaultRobotHWSim</robotSimType>
           <legacyModeNS>true</legacyModeNS>
+          <robotNamespace>$(arg ns)</robotNamespace>
         </plugin>
       </gazebo>
@@ -294,5 +294,5 @@
         <plugin name="sidebar_force_sensor" filename="libgazebo_ros_ft_sensor.so">
           <updateRate>100.0</updateRate>
-          <topicName>ft_sidebar</topicName>
+          <topicName>$(arg ns)/ft_sidebar</topicName>
           <jointName>joint_frame_hook</jointName>
           <noise>
@@ -306,5 +306,5 @@
         <plugin name="endeffector_force_sensor" filename="libgazebo_ros_ft_sensor.so">
           <updateRate>100.0</updateRate>
-          <topicName>ft_endeffector</topicName>
+          <topicName>$(arg ns)/ft_endeffector</topicName>
           <jointName>joint_vslider_hslider</jointName>
           <noise>
@@ -321,8 +321,8 @@
           </contact>
           <plugin name="gazebo_ros_bumper_controller" filename="libgazebo_ros_bumper.so">
-            <bumperTopicName>bumper_plug</bumperTopicName>
-            <frameName>world</frameName>
+            <bumperTopicName>$(arg ns)/bumper_plug</bumperTopicName>
+            <frameName>$(arg tf_prefix)/link_bp</frameName>
             <alwaysOn>true</alwaysOn>
-            <updateRate>5.0</updateRate>
+            <updateRate>100.0</updateRate>
           </plugin>
         </sensor>

File: ids_description/urdf/laser.urdf.xacro (robot description, xacro)
@@ -50,5 +50,5 @@
               <min>0.05</min>
               <max>30.0</max>
-              <resolution>0.01</resolution>
+              <resolution>0.001</resolution>
             </range>
             <noise>
@@ -59,6 +59,6 @@
           </ray>
           <plugin name="gazebo_ros_head_hokuyo_controller" filename="libgazebo_ros_gpu_laser.so">
-            <topicName>/laser/scan</topicName>
-            <frameName>link_hokuyo</frameName>
+            <topicName>$(arg ns)/laser/scan</topicName>
+            <frameName>$(arg tf_prefix)/link_hokuyo</frameName>
           </plugin>
         </sensor>
