Commit message: update parameters of navigation

File: ids_description/urdf/mrobot.urdf.xacro (robot description, xacro)
@@ -1,43 +1,45 @@
 <?xml version="1.0"?>
-<robot name="jazzy" xmlns:xacro="https://www.ros.org/wiki/xacro" >
-    <!--mobile base-->
-    <xacro:include filename="$(find ids_description)/urdf/base_square.urdf.xacro" />
-      <xacro:property name="mu" value="0.9"/>
-      <xacro:property name="mu2" value="0.7"/>
-    <xacro:fourwheeler_base_macro/>
-    <!--frame 3DOF-->
-    <xacro:include filename="$(find ids_description)/urdf/frame.urdf.xacro" />
-    <xacro:frame_macro parent="link_fbumper" name="mrobot">
-      <origin xyz="-0.11 0 0.14" rpy="0 0 0"/>
-    </xacro:frame_macro>
-    <!--RGB-D camera, look forward-->
-    <xacro:include filename="$(find ids_description)/urdf/realsense.urdf.xacro" />
-    <xacro:realsense_macro parent="link_hslider">
-      <xacro:property name="location_x" value="0.06"/>
-      <xacro:property name="location_y" value="0.0"/>
-      <xacro:property name="location_z" value="0.0725"/>
-      <xacro:property name="camera_width" value="640" />
-      <xacro:property name="camera_height" value="480" />
-      <xacro:property name="camera_name" value="camera" />
-    </xacro:realsense_macro>
-    <!--camera, look upward-->
-    <xacro:include filename="$(find ids_description)/urdf/camera.urdf.xacro"/>
-    <xacro:camera_macro parent="link_tip">
-      <xacro:property name="location_x" value="0.02" />
-      <xacro:property name="location_y" value="0.0" />
-      <xacro:property name="location_z" value="0.015" />
-      <xacro:property name="location_r" value="0" />
-      <xacro:property name="location_p" value="-1.57" />
-      <xacro:property name="location_y" value="0" />
-      <xacro:property name="camera_width" value="600" />
-      <xacro:property name="camera_height" value="600" />
-      <xacro:property name="camera_name" value="arducam"/>
-    </xacro:camera_macro>
-    <!-- laser -->
-    <xacro:include filename="$(find ids_description)/urdf/laser.urdf.xacro"/>
-    <xacro:laser_macro parent="link_fbumper">
-      <xacro:property name="location_x" value="0.05" />
-      <xacro:property name="location_y" value="0" />
-      <xacro:property name="location_z" value="0" />
-    </xacro:laser_macro>
+<robot name="mrobot" xmlns:xacro="https://www.ros.org/wiki/xacro">
+  <xacro:arg name="ns" default="" />
+  <xacro:arg name="tf_prefix" default=""/>
+  <!--mobile base-->
+  <xacro:include filename="$(find ids_description)/urdf/base_square.urdf.xacro" />
+    <xacro:property name="mu" value="0.98"/>
+    <xacro:property name="mu2" value="0.98"/>
+  <xacro:fourwheeler_base_macro/>
+  <!--frame 3DOF-->
+  <xacro:include filename="$(find ids_description)/urdf/frame.urdf.xacro" />
+  <xacro:frame_macro parent="link_fbumper">
+    <origin xyz="-0.11 0 0.14" rpy="0 0 0"/>
+  </xacro:frame_macro>
+  <!--RGB-D camera, look forward-->
+  <xacro:include filename="$(find ids_description)/urdf/realsense.urdf.xacro" />
+  <xacro:realsense_macro parent="link_hslider">
+    <xacro:property name="location_x" value="0.06"/>
+    <xacro:property name="location_y" value="0.0"/>
+    <xacro:property name="location_z" value="0.0725"/>
+    <xacro:property name="camera_width" value="640" />
+    <xacro:property name="camera_height" value="480" />
+    <xacro:property name="camera_name" value="camera" />
+  </xacro:realsense_macro>
+  <!--camera, look upward-->
+  <xacro:include filename="$(find ids_description)/urdf/camera.urdf.xacro"/>
+  <xacro:camera_macro parent="link_tip">
+    <xacro:property name="location_x" value="0.02" />
+    <xacro:property name="location_y" value="0.0" />
+    <xacro:property name="location_z" value="0.015" />
+    <xacro:property name="location_r" value="0" />
+    <xacro:property name="location_p" value="-1.57" />
+    <xacro:property name="location_y" value="0" />
+    <xacro:property name="camera_width" value="600" />
+    <xacro:property name="camera_height" value="600" />
+    <xacro:property name="camera_name" value="arducam"/>
+  </xacro:camera_macro>
+  <!-- laser -->
+  <xacro:include filename="$(find ids_description)/urdf/laser.urdf.xacro"/>
+  <xacro:laser_macro parent="link_fbumper">
+    <xacro:property name="location_x" value="0.05" />
+    <xacro:property name="location_y" value="0" />
+    <xacro:property name="location_z" value="0" />
+  </xacro:laser_macro>
 </robot>

File: ids_description/urdf/realsense.urdf.xacro (robot description, xacro)
@@ -65,5 +65,5 @@
           </camera>
           <plugin name="rs435_camera_plugin" filename="libgazebo_ros_openni_kinect.so">
-            <cameraName>${camera_name}</cameraName>
+            <cameraName>$(arg ns)/${camera_name}</cameraName>
             <imageTopicName>color/image_raw</imageTopicName>
             <cameraInfoTopicName>color/camera_info</cameraInfoTopicName>
@@ -71,5 +71,5 @@
             <depthImageCameraInfoTopicName>depth/camera_info</depthImageCameraInfoTopicName>
             <pointCloudTopicName>depth/points</pointCloudTopicName>
-            <frameName>rs435_frame</frameName>
+            <frameName>$(arg tf_prefix)/rs435_frame</frameName>
           </plugin>
         </sensor>

Commit message: update robot

File: ids_description/urdf/base_square.urdf.xacro (robot description, xacro)
@@ -224,5 +224,5 @@
     <!--baterry-->
     <joint name="joint_base_battery" type="fixed">
-      <origin xyz="0 0 ${base_z/2}" rpy="0 0 0"/>
+      <origin xyz="-0.1 0 ${base_z+battery_l/2}" rpy="0 0 0"/>
       <parent link="link_base"/>
       <child link="link_battery"/>
@@ -230,5 +230,5 @@
     <link name="link_battery">
       <visual>
-        <origin xyz="-0.15 0 0.08" rpy="0 0 0" />
+        <origin xyz="0 0 0" rpy="0 0 0" />
         <geometry>
           <box size="${battery_l} ${battery_l} ${battery_l}"/>
@@ -236,5 +236,5 @@
       </visual>
       <collision>
-        <origin xyz="-0.15 0 0.08" rpy="0 0 0" />
+        <origin xyz="0 0 0" rpy="0 0 0" />
         <geometry>
           <box size="${battery_l} ${battery_l} ${battery_l}"/>

File: ids_description/urdf/mrobot.urdf.xacro (robot description, xacro)
@@ -4,4 +4,6 @@
   <xacro:arg name="tf_prefix" default=""/>
   <!--mobile base-->
+  <!-- <xacro:include filename="$(find ids_description)/urdf/base_square.urdf.xacro" />
+  <xacro:fourwheeler_base_macro/> -->
   <xacro:include filename="$(find ids_description)/urdf/base_square.urdf.xacro" />
     <xacro:property name="mu" value="0.98"/>
@@ -17,6 +19,6 @@
     <xacro:property name="bumper_x" value="0.04" />
     <xacro:property name="bumper_y" value="0.52" />
-    <xacro:property name="battery_m" value="10" />
-    <xacro:property name="battery_l" value="0.3" />
+    <xacro:property name="battery_m" value="20" />
+    <xacro:property name="battery_l" value="0.5" />
   <xacro:fourwheeler_base_macro/>
   <!-- <xacro:include filename="$(find ids_description)/urdf/base_jazzy.urdf.xacro" />
