Commit message: change tip length in jrobot

File: ids_description/urdf/jframe.urdf.xacro (robot description, xacro)
@@ -194,13 +194,13 @@
       <link name="link_tip">
         <visual>
-          <origin rpy="0 0 0" xyz="0.01 0.01 0"/>
-          <geometry>
-            <box size="0.02 0.04 0.01"/>
-          </geometry>
-        </visual>
-        <collision>
-          <origin rpy="0 0 0" xyz="0.01 0.01 0"/>
-          <geometry>
-            <box size="0.02 0.04 0.01"/>
+          <origin rpy="0 0 0" xyz="0.01 0.02 0"/>
+          <geometry>
+            <box size="0.02 0.06 0.01"/>
+          </geometry>
+        </visual>
+        <collision>
+          <origin rpy="0 0 0" xyz="0.01 0.02 0"/>
+          <geometry>
+            <box size="0.02 0.06 0.01"/>
           </geometry>
         </collision>

File: ids_description/urdf/jrobot.urdf.xacro (robot description, xacro)
@@ -4,8 +4,5 @@
   <xacro:arg name="tf_prefix" default=""/>
   <xacro:include filename="$(find ids_description)/urdf/base_square.urdf.xacro" />
-  <xacro:fourwheeler_base_macro>
-    <xacro:property name="mu" value="0.9"/>
-    <xacro:property name="mu2" value="0.9"/>
-  </xacro:fourwheeler_base_macro>
+  <xacro:fourwheeler_base_macro/>
   <!--frame 3DOF-->
   <xacro:include filename="$(find ids_description)/urdf/jframe.urdf.xacro" />
