Commit message: add auto charge experiment

File: ids_description/urdf/camera.urdf.xacro (robot description, xacro)
@@ -29,5 +29,5 @@
         <origin xyz="0 0 ${camera_link/2}" rpy="0 0 0"/>
         <geometry>
-          <box size="${camera_link} ${camera_link} ${camera_link}"/>
+          <box size="${camera_link/2} ${camera_link} ${camera_link}"/>
         </geometry>
       </visual>
@@ -64,5 +64,5 @@
           <cameraName>/$(arg ns)/${camera_name}</cameraName>
           <imageTopicName>image</imageTopicName>
-          <cameraInfoTopicName>camera_info</cameraInfoTopicName>
+          <cameraInfoTopicName>cam_info</cameraInfoTopicName>
           <frameName>$(arg tf_prefix)/${camera_name}</frameName>
           <hackBaseline>0.07</hackBaseline>

File: ids_description/urdf/mrobot.urdf.xacro (robot description, xacro)
@@ -41,4 +41,16 @@
   <!--camera, look upward-->
   <xacro:include filename="$(find ids_description)/urdf/camera.urdf.xacro"/>
+  <xacro:camera_macro parent="link_hslider">
+    <xacro:property name="location_x" value="0.166" />
+    <xacro:property name="location_y" value="0.0" />
+    <xacro:property name="location_z" value="-0.05" />
+    <xacro:property name="location_r" value="0" />
+    <xacro:property name="location_p" value="0" />
+    <xacro:property name="location_y" value="0" />
+    <xacro:property name="camera_width" value="500" />
+    <xacro:property name="camera_height" value="500" />
+    <xacro:property name="camera_name" value="arducam1"/>
+  </xacro:camera_macro>
+  <xacro:include filename="$(find ids_description)/urdf/camera.urdf.xacro"/>
   <xacro:camera_macro parent="link_tip">
     <xacro:property name="location_x" value="0.02" />
@@ -48,7 +60,7 @@
     <xacro:property name="location_p" value="-1.57" />
     <xacro:property name="location_y" value="0" />
-    <xacro:property name="camera_width" value="600" />
-    <xacro:property name="camera_height" value="600" />
-    <xacro:property name="camera_name" value="arducam"/>
+    <xacro:property name="camera_width" value="500" />
+    <xacro:property name="camera_height" value="500" />
+    <xacro:property name="camera_name" value="arducam2"/>
   </xacro:camera_macro>
   <!-- laser -->

Commit message: refine code and remove duplicate code

File: ids_description/urdf/camera.urdf.xacro (robot description, xacro)
@@ -8,6 +8,6 @@
     <xacro:property name="location_p" value="0" />
     <xacro:property name="location_y" value="0" />
-    <xacro:property name="camera_width" value="600" />
-    <xacro:property name="camera_height" value="600" />
+    <xacro:property name="camera_width" value="400" />
+    <xacro:property name="camera_height" value="400" />
     <xacro:property name="camera_link" value="0.02" />
     <xacro:property name="camera_name" value="front_cam" />
@@ -56,5 +56,5 @@
             <type>gaussian</type>
             <mean>0.0</mean>
-            <stddev>0.007</stddev>
+            <stddev>0.001</stddev>
           </noise>
         </camera>
@@ -66,5 +66,5 @@
           <cameraInfoTopicName>cam_info</cameraInfoTopicName>
           <frameName>$(arg tf_prefix)/${camera_name}</frameName>
-          <hackBaseline>0.07</hackBaseline>
+          <hackBaseline>0.01</hackBaseline>
           <distortionK1>0.0</distortionK1>
           <distortionK2>0.0</distortionK2>

File: ids_description/urdf/mrobot.urdf.xacro (robot description, xacro)
@@ -39,5 +39,5 @@
     <xacro:property name="camera_name" value="camera" />
   </xacro:realsense_macro>
-  <!--camera, look upward-->
+  <!--2D camera, look forward-->
   <xacro:include filename="$(find ids_description)/urdf/camera.urdf.xacro"/>
   <xacro:camera_macro parent="link_hslider">
@@ -48,8 +48,9 @@
     <xacro:property name="location_p" value="0" />
     <xacro:property name="location_y" value="0" />
-    <xacro:property name="camera_width" value="500" />
-    <xacro:property name="camera_height" value="500" />
+    <xacro:property name="camera_width" value="400" />
+    <xacro:property name="camera_height" value="400" />
     <xacro:property name="camera_name" value="arducam1"/>
   </xacro:camera_macro>
+  <!--2D camera, look upward-->
   <xacro:include filename="$(find ids_description)/urdf/camera.urdf.xacro"/>
   <xacro:camera_macro parent="link_tip">
@@ -60,6 +61,6 @@
     <xacro:property name="location_p" value="-1.57" />
     <xacro:property name="location_y" value="0" />
-    <xacro:property name="camera_width" value="500" />
-    <xacro:property name="camera_height" value="500" />
+    <xacro:property name="camera_width" value="400" />
+    <xacro:property name="camera_height" value="400" />
     <xacro:property name="camera_name" value="arducam2"/>
   </xacro:camera_macro>

Commit message: change camera fov

File: ids_description/urdf/camera.urdf.xacro (robot description, xacro)
@@ -8,6 +8,6 @@
     <xacro:property name="location_p" value="0" />
     <xacro:property name="location_y" value="0" />
-    <xacro:property name="camera_width" value="400" />
-    <xacro:property name="camera_height" value="400" />
+    <xacro:property name="camera_width" value="500" />
+    <xacro:property name="camera_height" value="500" />
     <xacro:property name="camera_link" value="0.02" />
     <xacro:property name="camera_name" value="front_cam" />
@@ -43,5 +43,5 @@
         <update_rate>30.0</update_rate>
         <camera name="head">
-          <horizontal_fov>1.3962634</horizontal_fov>
+          <horizontal_fov>0.61</horizontal_fov>
           <image>
             <width>${camera_width}</width>
@@ -61,5 +61,5 @@
         <plugin name="camera_controller" filename="libgazebo_ros_camera.so">
           <alwaysOn>true</alwaysOn>
-          <updateRate>60</updateRate>
+          <updateRate>30</updateRate>
           <cameraName>/$(arg ns)/${camera_name}</cameraName>
           <imageTopicName>image</imageTopicName>

File: ids_description/urdf/jframe.urdf.xacro (robot description, xacro)
@@ -154,5 +154,5 @@
       <!--hook for door opening-->
       <joint name="joint_frame_hook" type="revolute">
-        <origin xyz="0.31 -0.23 0.3" rpy="0 0 0"/>
+        <origin xyz="0.31 -0.23 0.05" rpy="0 0 0"/>
         <parent link="link_frame"/>
         <child link="link_hook"/>

File: ids_description/urdf/mrobot.urdf.xacro (robot description, xacro)
@@ -9,5 +9,5 @@
   <xacro:include filename="$(find ids_description)/urdf/frame.urdf.xacro" />
   <xacro:frame_macro parent="link_fbumper">
-    <origin xyz="-0.11 0 0.14" rpy="0 0 0"/>
+    <origin xyz="-0.11 0 0.15" rpy="0 0 0"/>
   </xacro:frame_macro>
   <!--RGB-D camera, look forward-->
@@ -30,6 +30,6 @@
     <xacro:property name="location_p" value="0" />
     <xacro:property name="location_y" value="0" />
-    <xacro:property name="camera_width" value="400" />
-    <xacro:property name="camera_height" value="400" />
+    <xacro:property name="camera_width" value="500" />
+    <xacro:property name="camera_height" value="500" />
     <xacro:property name="camera_name" value="arducam1"/>
   </xacro:camera_macro>
@@ -43,6 +43,6 @@
     <xacro:property name="location_p" value="-1.57" />
     <xacro:property name="location_y" value="0" />
-    <xacro:property name="camera_width" value="400" />
-    <xacro:property name="camera_height" value="400" />
+    <xacro:property name="camera_width" value="500" />
+    <xacro:property name="camera_height" value="500" />
     <xacro:property name="camera_name" value="arducam2"/>
   </xacro:camera_macro>
