Commit message: refine plugin

File: ids_description/urdf/mrobot.urdf.xacro (robot description, xacro)
@@ -44,5 +44,5 @@
     <xacro:property name="location_x" value="0.166" />
     <xacro:property name="location_y" value="0.0" />
-    <xacro:property name="location_z" value="-0.05" />
+    <xacro:property name="location_z" value="-0.04" />
     <xacro:property name="location_r" value="0" />
     <xacro:property name="location_p" value="0" />

Commit message: update tests

File: ids_description/urdf/mrobot.urdf.xacro (robot description, xacro)
@@ -9,5 +9,5 @@
   <xacro:include filename="$(find ids_description)/urdf/frame.urdf.xacro" />
   <xacro:frame_macro parent="link_fbumper">
-    <origin xyz="-0.11 0 0.15" rpy="0 0 0"/>
+    <origin xyz="-0.11 0 0.14" rpy="0 0 0"/>
   </xacro:frame_macro>
   <!--RGB-D camera, look forward-->
