Commit message: change joint position of sidebar

File: ids_description/urdf/jframe_r.urdf.xacro (robot description, xacro)
@@ -154,5 +154,5 @@
       <!--hook for door opening-->
       <joint name="joint_frame_hook" type="revolute">
-        <origin xyz="0.31 -0.23 0.05" rpy="0 0 0"/>
+        <origin xyz="0.165 -0.23 0.05" rpy="0 0 0"/>
         <parent link="link_frame"/>
         <child link="link_hook"/>
@@ -162,5 +162,5 @@
       <link name="link_hook">
         <visual>
-          <origin rpy="0 0 0" xyz="0 0 0"/>
+          <origin rpy="0 0 0" xyz="0.145 0 0"/>
           <geometry>
             <box size="0.4 0.02 0.01"/>
@@ -168,5 +168,5 @@
         </visual>
         <collision>
-          <origin rpy="0 0 0" xyz="0 0 0"/>
+          <origin rpy="0 0 0" xyz="0.145 0 0"/>
           <geometry>
             <box size="0.4 0.02 0.01"/>
@@ -188,5 +188,5 @@
       </link>
       <joint name="joint_hook_tip" type="fixed">
-        <origin xyz="0.2 0 0" rpy="0 0 0"/>
+        <origin xyz="0.345 0 0" rpy="0 0 0"/>
         <parent link="link_hook"/>
         <child link="link_tip"/>
